File: bee-inamp.sch (KiCad schematic (older format))
At the start: 4 parts, among them J1 Conn_01x02_Male, J2 Conn_01x02_Male, J3 Conn_01x02_Male, J4 Conn_01x02_Male

Commit message: schematic and layout
Parts:
- added C1, C2: 0.1µF, Capacitor_SMD:C_0805_2012Metric_Pad1.15x1.40mm_HandSolder, symbol Device:C
- added J5, J6: Conn_01x02, Connector_PinSocket_2.54mm:PinSocket_1x02_P2.54mm_Vertical, symbol Connector_Generic:Conn_01x02
- added J7: Conn_02x03_Odd_Even, Connector_PinHeader_2.54mm:PinHeader_2x03_P2.54mm_Vertical_SMD, symbol Connector_Generic:Conn_02x03_Odd_Even
- added J8: Conn_01x03, Connector_PinHeader_2.54mm:PinHeader_1x03_P2.54mm_Vertical, symbol Connector_Generic:Conn_01x03
- added J9: Conn_01x02, Connector_PinHeader_2.54mm:PinHeader_1x02_P2.54mm_Vertical, symbol Connector_Generic:Conn_01x02
- added JP1: SolderJumper_2_Bridged, Jumper:SolderJumper-2_P1.3mm_Bridged_Pad1.0x1.5mm, symbol Jumper:SolderJumper_2_Bridged
- added R1: 16k, Resistor_SMD:R_0805_2012Metric_Pad1.15x1.40mm_HandSolder, symbol Device:R
- added R2: 820R, Resistor_SMD:R_0805_2012Metric_Pad1.15x1.40mm_HandSolder, symbol Device:R
- added U1: INA126, Package_SO:SO-8_5.3x6.2mm_P1.27mm, symbol Amplifier_Instrumentation:INA128
Connections:
- net +15V: now also C1.1, U1.7 (V+)
- net -15V: now also C2.1, U1.4 (V-)
- net GND: now also C1.2, C2.2, J8.2 (Pin_2), J9.2 (Pin_2), JP1.2 (B)
- new net: JP1.1 (A), U1.5 (Ref)
- new net: J9.1 (Pin_1), U1.6
- new net: J7.1 (Pin_1), R1.1
- new net: J7.3 (Pin_3), R2.1
- new net: J6.1 (Pin_1), J6.2 (Pin_2), J7.5 (Pin_5)
- new net Rg_1: J7.2 (Pin_2), J7.4 (Pin_4), J7.6 (Pin_6), U1.1 (Rg)
- new net Rg_2: J5.1 (Pin_1), J5.2 (Pin_2), R1.2, R2.2, U1.8 (Rg)
- new net in+: J8.1 (Pin_1), U1.3 (+)
- new net in-: J8.3 (Pin_3), U1.2 (-)
Other:
- note added: "G = 10"
- note added: "G = 100"
- note added: "G = variabel \nper Widerstand, bedrahtet"
